File: pcb/pcb.kicad_sch (KiCad schematic)
At the start: 12 parts, among them CN1 1x3, CN2 1x8, CN3 1x8, CN4 1x8, CN5 1x4, CN6 1x2, CN7 1x2, SW1 switch_3x4, SW2 switch_3x4

Commit message: merge
Parts:
- added CN8: ~, USB:USB4105-GF-A, symbol connectors:USB4105-GF-A
- added R12, R13: 5k1, SMT:0603, symbol generic:R
Connections:
- net GND: now also CN8.A1 (GND), CN8.A4 (VBUS), CN8.B1 (GND), CN8.B4 (VBUS), CN8.S1 (SHLD), CN8.S2 (SHLD), CN8.S3 (SHLD), CN8.S4 (SHLD), R12.2, R13.2
- net MCU/USB_M: now also CN8.A7 (D1N), CN8.B7 (DN2)
- net MCU/USB_P: now also CN8.A6 (D1P), CN8.B6 (DP2)
- new net: CN8.A5 (CC1), R13.1
- new net: CN8.B5 (CC2), R12.1
